Commit message: Add files via upload

File: urdf/wheelchair_xarm.urdf (robot description, URDF)
Before this commit: robot wheelchair_with_xarm7, 34 links, 33 joints
Links:
- removed link laser_left
- removed link laser_right
Joints:
- removed joint lidar_left_joint
- removed joint lidar_right_joint
- joint BL_joint: axis 0 1 0 -> (none); limit effort=150.0 velocity=10.0 -> (none); type continuous -> fixed
- joint BR_joint: axis 0 1 0 -> (none); limit effort=150.0 velocity=10.0 -> (none); type continuous -> fixed
- joint FL_joint: axis 0 1 0 -> (none); type continuous -> fixed
- joint FR_joint: axis 0 1 0 -> (none); type continuous -> fixed
