Commit message: update urdf path to mesh

File: urdf/wheelchair_spherized_foam.urdf (robot description, URDF)
Before this commit: robot wheelchair, 26 links, 25 joints
Links:
- link back_left_1: geometry collision sphere radius=0.125902; visual mesh filename=package://wheelchair_xarm/meshes/wheelchair/back.stl scale=0.001 0.001 0.001
- link back_right_1: geometry collision sphere radius=0.135849; visual mesh filename=package://wheelchair_xarm/meshes/wheelchair/back.stl scale=0.001 0.001 0.001
- link base_link: geometry collision sphere radius=0.033547; collision sphere radius=0.033864
- link front_left_1: geometry collision sphere radius=0.135528; collision sphere radius=0.135648
- link front_right_1: geometry collision sphere radius=0.126117; collision sphere radius=0.127501
- link left_finger: geometry collision sphere radius=0.023718; collision sphere radius=0.024779
- link left_inner_knuckle: geometry collision sphere radius=0.020015; collision sphere radius=0.021056
- link left_outer_knuckle: geometry collision sphere radius=0.016872; collision sphere radius=0.0173
- link link1: geometry collision sphere radius=0.08051; collision sphere radius=0.082405
- link link2: geometry collision sphere radius=0.05706; collision sphere radius=0.059383
- link link3: geometry collision sphere radius=0.057955; collision sphere radius=0.060511
- link link4: geometry collision sphere radius=0.049704; collision sphere radius=0.052523
- link link5: geometry collision sphere radius=0.047642; collision sphere radius=0.060203
- link link6: geometry collision sphere radius=0.053225; collision sphere radius=0.053291
- link link7: geometry collision sphere radius=0.029515; collision sphere radius=0.040936
- link link_base: geometry collision sphere radius=0.087042; collision sphere radius=0.095256
- link link_eef: geometry collision sphere radius=0.0284; collision sphere radius=0.03107
- link right_finger: geometry collision sphere radius=0.023204; collision sphere radius=0.025204
- link right_inner_knuckle: geometry collision sphere radius=0.020151; collision sphere radius=0.020278
- link right_outer_knuckle: geometry collision sphere radius=0.017545; collision sphere radius=0.017688
- link xarm_gripper_base_link: geometry collision sphere radius=0.072277; visual mesh filename=package://wheelchair_xarm/meshes/gripper/xarm/base_link.stl
